File: Hardware/file55955BF9.sch (KiCad schematic (older format))
At the start: 45 parts, among them P201 CONN_01X02, Q201 CSD18532Q5B, Q202 CSD18532Q5B, U201 TPS40054

Commit message: Platine bis auf Sicherung fertig
Parts:
- removed R215: 0*, Resistors_SMD:R_0603, symbol R
- added P3, P4, P5, P6: CONN_01X01, Mounting_Holes:MountingHole_3mm, symbol CONN_01X01
- gave numbers to parts that had none: 3
Connections:
- net GND: now also R216.1
- net GNDREF: no longer R216.1
- no-connect marks 0 -> 4
Other:
- note added: "Befestigungslöcher M3"
