File: Hardware/file55A12ABE.sch (KiCad schematic (older format))
At the start: 7 parts, among them P301 CONN_01X06, P302 CONN_01X06, P303 CONN_01X08, P304 CONN_01X08, Q301 BC807-40

Commit message: Schaltplan momentan fertig - Netzliste angefangen.
Parts:
- C301: footprint Capacitors_SMD:C_0402 -> Capacitors_SMD:C_0603
- P301, P302: footprint (none) -> Pin_Headers:Pin_Header_Straight_1x06
- P303, P304: footprint (none) -> Pin_Headers:Pin_Header_Straight_1x08
- Q301: footprint SOT-23 -> Housings_SOT-23_SOT-143_TSOT-6:SOT-23
Changed lines of the file:
@@
 LIBS:w_microcontrollers
 LIBS:ph-diodes
+LIBS:ph-sensor
 LIBS:stm32 APRS Tracker-cache
 EELAYER 25 0
@@
 F 0 "P301" H 5700 3800 50  0000 C CNN
 F 1 "CONN_01X06" V 5800 3450 50  0000 C CNN
-F 2 "" H 5700 3450 60  0000 C CNN
+F 2 "Pin_Headers:Pin_Header_Straight_1x06" H 5700 3450 60  0001 C CNN
 F 3 "" H 5700 3450 60  0000 C CNN
 	1    5700 3450
@@
 F 0 "P302" H 5700 4700 50  0000 C CNN
 F 1 "CONN_01X06" V 5800 4350 50  0000 C CNN
-F 2 "" H 5700 4350 60  0000 C CNN
+F 2 "Pin_Headers:Pin_Header_Straight_1x06" H 5700 4350 60  0001 C CNN
 F 3 "" H 5700 4350 60  0000 C CNN
 	1    5700 4350
@@
 F 0 "P304" H 6500 4700 50  0000 C CNN
 F 1 "CONN_01X08" V 6600 4250 50  0000 C CNN
-F 2 "" H 6500 4250 60  0000 C CNN
+F 2 "Pin_Headers:Pin_Header_Straight_1x08" H 6500 4250 60  0001 C CNN
 F 3 "" H 6500 4250 60  0000 C CNN
 	1    6500 4250
@@
 F 0 "P303" H 6500 3600 50  0000 C CNN
 F 1 "CONN_01X08" V 6600 3150 50  0000 C CNN
-F 2 "" H 6500 3150 60  0000 C CNN
+F 2 "Pin_Headers:Pin_Header_Straight_1x08" H 6500 3150 60  0001 C CNN
 F 3 "" H 6500 3150 60  0000 C CNN
 	1    6500 3150
@@
 Reset
 $Comp
-L +3.3V #PWR0106
+L +3.3V #PWR0116
 U 1 1 55A21974
 P 5500 3300
-F 0 "#PWR0106" H 5500 3150 50  0001 C CNN
+F 0 "#PWR0116" H 5500 3150 50  0001 C CNN
 F 1 "+3.3V" H 5500 3440 50  0000 C CNN
 F 2 "" H 5500 3300 60  0000 C CNN
@@
 $EndComp
 $Comp
-L GND #PWR0107
+L GND #PWR0117
 U 1 1 55A219AE
 P 5500 3500
-F 0 "#PWR0107" H 5500 3250 50  0001 C CNN
+F 0 "#PWR0117" H 5500 3250 50  0001 C CNN
 F 1 "GND" H 5500 3350 50  0000 C CNN
 F 2 "" H 5500 3500 60  0000 C CNN
@@
 $EndComp
 $Comp
-L GND #PWR0108
+L GND #PWR0118
 U 1 1 55A21C31
 P 5500 3600
-F 0 "#PWR0108" H 5500 3350 50  0001 C CNN
+F 0 "#PWR0118" H 5500 3350 50  0001 C CNN
 F 1 "GND" H 5500 3450 50  0000 C CNN
 F 2 "" H 5500 3600 60  0000 C CNN
@@
 $EndComp
 $Comp
-L +3.3V #PWR0109
+L +3.3V #PWR0119
 U 1 1 55A21C48
 P 5500 3700
-F 0 "#PWR0109" H 5500 3550 50  0001 C CNN
+F 0 "#PWR0119" H 5500 3550 50  0001 C CNN
 F 1 "+3.3V" H 5500 3840 50  0000 C CNN
 F 2 "" H 5500 3700 60  0000 C CNN
@@
 F 0 "Q301" H 4900 3075 50  0000 L CNN
 F 1 "BC807-40" H 4900 3000 50  0000 L CNN
-F 2 "SOT-23" H 4900 2925 50  0000 L CIN
+F 2 "Housings_SOT-23_SOT-143_TSOT-6:SOT-23" H 4900 2925 50  0000 L CIN
 F 3 "" H 4700 3000 50  0000 L CNN
 	1    4700 3000
@@
 F 0 "C301" H 4825 3650 50  0000 L CNN
 F 1 "100n" H 4825 3450 50  0000 L CNN
-F 2 "Capacitors_SMD:C_0402" H 4838 3400 30  0001 C CNN
+F 2 "Capacitors_SMD:C_0603" H 4838 3400 30  0001 C CNN
 F 3 "" H 4800 3550 60  0000 C CNN
 	1    4800 3550
@@
 $EndComp
 $Comp
-L GND #PWR0110
+L GND #PWR0120
 U 1 1 55A21D74
 P 4800 3700
-F 0 "#PWR0110" H 4800 3450 50  0001 C CNN
+F 0 "#PWR0120" H 4800 3450 50  0001 C CNN
 F 1 "GND" H 4800 3550 50  0000 C CNN
 F 2 "" H 4800 3700 60  0000 C CNN
@@
 	4800 3400 4800 3200
 $Comp
-L +3.3V #PWR0111
+L +3.3V #PWR0121
 U 1 1 55A21DE4
 P 4800 2800
-F 0 "#PWR0111" H 4800 2650 50  0001 C CNN
+F 0 "#PWR0121" H 4800 2650 50  0001 C CNN
 F 1 "+3.3V" H 4800 2940 50  0000 C CNN
 F 2 "" H 4800 2800 60  0000 C CNN
